File: Schematic/Joystick_Schematic/Joystick_Schematic.kicad_sch (KiCad schematic)
At the start: 25 parts, among them SW2 SKQUCAA010, SW3 SKQUCAA010, U1 74HC165, U2 ATmega328P-A, U3 74HC165, U4 74HC165, U5 CH340G

Commit message: Finished Faceplate-PCB
Parts:
- J1: value (none) -> Conn_01x06_Female; footprint (none) -> Connector_PinSocket_2.54mm:PinSocket_1x06_P2.54mm_Vertical
- J2: value (none) -> Conn_01x04_Female; footprint (none) -> Connector_PinSocket_2.54mm:PinSocket_1x04_P2.54mm_Vertical
- J3: value (none) -> Conn_01x02_Female; footprint (none) -> Connector_PinSocket_2.54mm:PinSocket_1x02_P2.54mm_Vertical
- RN1, RN2, RN3, RN4, RN5, RN6: value (none) -> 1k; footprint (none) -> Resistor_THT:R_Array_SIP5
- RV1: value (none) -> RKJXV122400R; footprint (none) -> Alps-RKJXV:RKJXV122400R
- SW1: value (none) -> RKJXT1F42001
Other:
- moved on the sheet: RV1
