File: Schematic/Sub-Controller-PCB/Sub-Controller-PCB.kicad_pcb (KiCad board)
At the start: 2 copper layers, 40.6 x 25.4 mm, 2 parts, among them J1 Conn_01x03_Female, J2 Conn_01x04_Female

Commit message: started working on Sub-Controller-PCB
Parts:
- added C1: 100nF, Resistor_SMD:R_0201_0603Metric_Pad0.64x0.40mm_HandSolder, B.Cu at (144.8, 89.3)
- added C2: 100nF, Resistor_SMD:R_0201_0603Metric_Pad0.64x0.40mm_HandSolder, B.Cu at (137.8, 97.8)
- added J3: Conn_01x04_Female, Connector_PinSocket_2.54mm:PinSocket_1x04_P2.54mm_Vertical, F.Cu at (135.3, 89.5)
- added J4: Conn_01x02_Female, Connector_PinSocket_2.54mm:PinSocket_1x02_P2.54mm_Vertical, F.Cu at (151.2, 90.8)
- added J5: Conn_01x04_Female, Connector_PinSocket_2.54mm:PinSocket_1x04_P2.54mm_Vertical, F.Cu at (189.5, 115.8)
- added J6: Conn_01x04_Female, Connector_PinSocket_2.54mm:PinSocket_1x04_P2.54mm_Vertical, F.Cu at (167.3, 108.2)
- added J7: Conn_01x04_Female, Connector_PinSocket_2.54mm:PinSocket_1x04_P2.54mm_Vertical, F.Cu at (151.1, 125.1)
- added J8: Conn_01x04_Female, Connector_PinSocket_2.54mm:PinSocket_1x04_P2.54mm_Vertical, F.Cu at (130.2, 124.4)
- added JUSB1: USB_B_Micro, Connector_USB:USB_Micro-B_Molex_47346-0001, B.Cu at (144.1, 71.8)
- added RN1: 1k, Resistor_SMD:R_Array_Convex_4x1206, F.Cu at (171.7, 112.0)
- added RN2: 1k, Resistor_SMD:R_Array_Convex_4x1206, F.Cu at (185.1, 112.0)
- added RN3: 1k, Resistor_SMD:R_Array_Convex_4x1206, F.Cu at (153.0, 120.0)
- added RN4: 1k, Resistor_SMD:R_Array_Convex_4x1206, F.Cu at (136.5, 120.0)
- added RP1A1: 1k, Resistor_SMD:R_0201_0603Metric_Pad0.64x0.40mm_HandSolder, B.Cu at (149.9, 82.8)
- added RP1B1: 1k, Resistor_SMD:R_0201_0603Metric_Pad0.64x0.40mm_HandSolder, B.Cu at (148.6, 82.1)
- added U1: ATmega328P-A, Package_QFP:TQFP-32_7x7mm_P0.8mm, B.Cu at (144.1, 97.8)
- added U2: 74HC165, Package_SO:TSSOP-16_4.4x5mm_P0.65mm, F.Cu at (178.4, 111.8)
- added U3: 74HC165, Package_SO:TSSOP-16_4.4x5mm_P0.65mm, F.Cu at (144.8, 120.7)
- added U4: CH340G, Package_SO:SOIC-16_3.9x9.9mm_P1.27mm, B.Cu at (144.1, 81.3)
- J1: value Conn_01x03_Female -> Conn_01x03_Male; footprint Connector_PinHeader_2.54mm:PinHeader_1x03_P2.54mm_Vertical -> Connector_PinSocket_2.54mm:PinSocket_1x03_P2.54mm_Vertical
- J2: value Conn_01x04_Female -> Conn_01x04_Male; footprint Connector_PinHeader_2.54mm:PinHeader_1x04_P2.54mm_Vertical -> Connector_PinSocket_2.54mm:PinSocket_1x04_P2.54mm_Vertical
Connections:
- J1 pad 1: (no net) -> /SH_LATCH
- J1 pad 2: (no net) -> /SH_CLK
- J1 pad 3: (no net) -> /SH_DATA1
- J2 pad 1: (no net) -> GND
- J2 pad 2: (no net) -> +5V
- J2 pad 3: (no net) -> /HAT2_PUSH
- J2 pad 4: (no net) -> /HAT1_PUSH
Routing:
- net /SH_DATA1: track 0.00 -> 30.5 mm
- net GND: track 0.00 -> 20.4 mm
- net /SH_LATCH: track 0.00 -> 18.6 mm
- net /SH_CLK: track 0.00 -> 17.8 mm
- net Net-(RP1A1-Pad1): track 0.00 -> 12.3 mm, vias 0 -> 2
- net Net-(RP1B1-Pad1): track 0.00 -> 12.0 mm
- net Net-(JUSB1-Pad2): track 0.00 -> 11.5 mm
- net Net-(JUSB1-Pad3): track 0.00 -> 9.95 mm
- net Net-(C1-Pad1): track 0.00 -> 9.79 mm
- net /THUMB_X: track 0.00 -> 8.75 mm
- net /THUMB_Y: track 0.00 -> 6.91 mm
- net /RX: track 0.00 -> 5.80 mm
- net /ENCODER_A: track 0.00 -> 5.33 mm
- net /SDA: track 0.00 -> 5.11 mm
- net /SCL: track 0.00 -> 4.39 mm
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Other:
- board size 40.6 x 25.4 mm -> 40.6 x 41.3 mm

Commit message: Finished preliminary routing of sub-controller pcb
Parts:
- moved RN1 42.9 mm to (132.3, 94.9)
- moved RN2 42.9 mm to (145.7, 94.9)
- moved U2 42.9 mm to (139.1, 94.6)
- moved J6 42.5 mm to (128.3, 91.4)
- moved J5 40.9 mm to (154.9, 94.0)
- moved J7 34.2 mm to (160.0, 92.1), turned to 0 degrees
- moved U3 19.8 mm to (142.9, 101.0)
- moved RN3 19.7 mm to (153.7, 100.3)
- moved RN4 17.3 mm to (131.4, 103.5)
- moved J8 16.9 mm to (126.4, 107.9)
Connections:
- J6 pad 4: /NC -> /RESERVED1
- J8 pad 2: /NC -> /RESERVED2
- RN1 pad 1: /NC -> /RESERVED1
- RN4 pad 2: /NC -> /RESERVED2
- U2 pad 6: /NC -> /RESERVED1
- U3 pad 4: /NC -> /RESERVED2
Routing:
- net GND: track 20.4 -> 127.1 mm, vias 0 -> 7
- net +5V: track 4.11 -> 92.0 mm, vias 0 -> 5
- net /RESERVED2: track 0.00 -> 32.4 mm, vias 0 -> 1
- net /SH_CLK: track 17.8 -> 47.8 mm, vias 0 -> 2
- net /SH_LATCH: track 18.6 -> 44.7 mm, vias 0 -> 3
- net /THUMB_PUSH: track 0.00 -> 21.3 mm, vias 0 -> 2
- net /TRIGGER_1: track 0.00 -> 20.4 mm, vias 0 -> 2
- net /HAT2_PUSH: track 0.00 -> 19.5 mm
- net /TRIGGER_2: track 0.00 -> 19.4 mm, vias 0 -> 2
- net /TOP_SIDE_PUSH: track 0.00 -> 18.9 mm
- net /RKJXT1F_DOWN: track 0.00 -> 18.2 mm
- net /RKJXT1F_LEFT: track 0.00 -> 17.9 mm
- net /HAT1_PUSH: track 0.00 -> 17.8 mm
- net /RKJXT1F_UP: track 0.00 -> 17.3 mm
- net /PANEL_PUSH: track 0.00 -> 16.7 mm
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
Commit message: small modifications to to sub-controller-pcb
Parts:
- moved RN3 1.30 mm to (155.0, 100.3)
Routing:
- net /THUMB_PUSH: track 21.3 -> 27.8 mm, vias 2 -> 0
- net /TRIGGER_1: track 20.4 -> 25.1 mm, vias 2 -> 0
- net /TRIGGER_2: track 19.4 -> 21.6 mm, vias 2 -> 0

Commit message: PCB rework
Parts:
- removed JUSB1: USB_B_Micro, Connector_USB:USB_Micro-B_Molex_47346-0001
- added C3: 100nF, Capacitor_SMD:C_0603_1608Metric_Pad1.08x0.95mm_HandSolder, B.Cu at (141.2, 95.6)
- added C4: 100nF, Capacitor_SMD:C_0603_1608Metric_Pad1.08x0.95mm_HandSolder, B.Cu at (144.3, 94.6)
- added C5: 100nF, Capacitor_SMD:C_0603_1608Metric_Pad1.08x0.95mm_HandSolder, B.Cu at (141.2, 92.0)
- added C6: 100nF, Capacitor_SMD:C_0603_1608Metric_Pad1.08x0.95mm_HandSolder, F.Cu at (142.7, 70.4)
- added J10: Conn_01x04_Female, Connector_PinSocket_2.54mm:PinSocket_1x04_P2.54mm_Vertical, F.Cu at (147.6, 70.4)
- added J9: Conn_01x02_Female, Connector_PinSocket_2.54mm:PinSocket_1x02_P2.54mm_Vertical, F.Cu at (156.5, 89.9)
- added R1: 4.7k, Resistor_SMD:R_0603_1608Metric_Pad0.98x0.95mm_HandSolder, F.Cu at (153.7, 89.8)
- C1, RP1A1, RP1B1: footprint Resistor_SMD:R_0201_0603Metric_Pad0.64x0.40mm_HandSolder -> Resistor_SMD:R_0603_1608Metric_Pad0.98x0.95mm_HandSolder; moved to F.Cu
- C2: footprint Resistor_SMD:R_0201_0603Metric_Pad0.64x0.40mm_HandSolder -> Capacitor_SMD:C_0603_1608Metric_Pad1.08x0.95mm_HandSolder
- RN1, RN2, RN3: moved to B.Cu
- U1: moved to F.Cu
- moved J6 29.8 mm to (155.7, 103.1), turned to -90 degrees
- moved RN3 25.4 mm to (130.3, 94.2)
- moved J7 24.2 mm to (135.9, 90.2), turned to -90 degrees
- moved RN1 20.1 mm to (152.4, 95.2), turned to 0 degrees
- moved U2 15.5 mm to (154.4, 96.5)
- moved J3 15.4 mm to (150.6, 91.2), turned to 180 degrees
- moved C1 13.7 mm to (142.2, 75.8)
- moved U3 13.4 mm to (130.3, 96.3), turned to 90 degrees
- moved J4 11.7 mm to (141.2, 84.6), turned to 180 degrees
- moved RN2 11.3 mm to (157.0, 95.2), turned to 180 degrees
- moved C2 8.62 mm to (145.8, 94.6)
- moved J5 7.74 mm to (160.8, 99.1)
- moved U4 7.50 mm to (142.7, 73.9)
- moved J8 7.27 mm to (131.8, 103.1)
- moved RN4 5.64 mm to (126.0, 104.9), turned to 0 degrees
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Routing:
- net GND: track 127.1 -> 152.6 mm, vias 7 -> 9
- net /HAT2_PUSH: track 19.5 -> 40.2 mm
- net /THUMB_PUSH: track 27.8 -> 9.14 mm, vias 0 -> 1
- net /HAT1_PUSH: track 17.8 -> 36.1 mm
- net /TRIGGER_1: track 25.1 -> 6.96 mm, vias 0 -> 1
- net /TRIGGER_2: track 21.6 -> 6.04 mm, vias 0 -> 1
- net /SH_DATA1: track 36.1 -> 22.2 mm
- net /TX: track 3.40 -> 16.0 mm, vias 0 -> 1
- net /RKJXT1F_DOWN: track 18.2 -> 6.18 mm
- net /RESET: track 3.90 -> 15.2 mm, vias 0 -> 2
- net +5V: track 92.1 -> 103.3 mm
- net /RKJXT1F_LEFT: track 17.9 -> 6.97 mm
- net /PANEL_PUSH: track 17.0 -> 6.40 mm, vias 0 -> 1
- net /RKJXT1F_UP: track 17.3 -> 7.20 mm
- net /RX: track 5.80 -> 14.8 mm, vias 0 -> 1
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
Commit message: Some PCB changes
Parts:
- added C7: 4.7nF, Capacitor_SMD:C_0603_1608Metric_Pad1.08x0.95mm_HandSolder, F.Cu at (144.8, 73.0)
- U4: value CH340G -> CH340C
Connections:
- C6 pad 1: +5V -> Net-(C6-Pad1)
- J10 pad 4: +5V -> Net-(C6-Pad1)
- U4 pad 16: +5V -> Net-(C6-Pad1)
- U4 pad 4: unconnected-(U4-Pad4) -> Net-(C7-Pad2)
Routing:
- net +5V: track 103.3 -> 75.1 mm, vias 5 -> 4
- net Net-(C6-Pad1): track 0.00 -> 15.7 mm, vias 0 -> 1
- net GND: track 152.6 -> 155.7 mm
- net Net-(C7-Pad2): track 0.00 -> 2.09 mm, vias 0 -> 1
