File: Schematic/Sub-Controller-PCB/Sub-Controller-PCB.kicad_sch (KiCad schematic)
At the start: 2 parts

Commit message: started working on Sub-Controller-PCB
Parts:
- added C1: (no value), symbol Device:C
- added C2: 100nF, Resistor_SMD:R_0201_0603Metric_Pad0.64x0.40mm_HandSolder, symbol Device:C
- added J3, J5, J6, J7, J8: (no value), symbol Connector:Conn_01x04_Female
- added J4: (no value), symbol Connector:Conn_01x02_Female
- added JUSB1: (no value), symbol Connector:USB_B_Micro
- added RN1, RN2, RN3, RN4: (no value), symbol Device:R_Pack04
- added RP1A1: (no value), symbol Device:R
- added RP1B1: 1k, Resistor_SMD:R_0201_0603Metric_Pad0.64x0.40mm_HandSolder, symbol Device:R
- added U1: (no value), symbol MCU_Microchip_ATmega:ATmega328P-A
- added U2, U3: (no value), symbol 74xx:74HC165
- added U4: CH340G, Package_SO:SOIC-16_3.9x9.9mm_P1.27mm, symbol Interface_USB:CH340G
Connections:
- net SH_LATCH: now reaches J1.1 (Pin_1)
- net SH_LATCH: now also U1.24 (PC1), U2.1 (~{PL}), U3.1 (~{PL})
- net SH_CLK: now reaches J1.2 (Pin_2)
- net SH_CLK: now also U1.23 (PC0), U2.2 (CP), U3.2 (CP)
- net SH_DATA1: now reaches J1.3 (Pin_3)
- net SH_DATA1: now also U1.12 (PB0)
- net GND: now reaches J2.1 (Pin_1)
- net GND: now also C2.2, JUSB1.5 (GND), JUSB1.6 (Shield), RN1.5 (R4.2), RN1.6 (R3.2), RN1.7 (R2.2), RN1.8 (R1.2), RN2.5 (R4.2), RN2.6 (R3.2), RN2.7 (R2.2), RN2.8 (R1.2), RN3.5 (R4.2), RN3.6 (R3.2), RN3.7 (R2.2), RN3.8 (R1.2), RN4.5 (R4.2), RN4.6 (R3.2), RN4.7 (R2.2), RN4.8 (R1.2), U1.21 (GND), U1.3 (GND), U1.5 (GND), U2.10 (DS), U2.15 (~{CE}), U2.8 (GND), U3.10 (DS), U3.15 (~{CE}), U3.8 (GND), U4.1 (GND)
- net +5V: now reaches J2.2 (Pin_2)
- net +5V: now also JUSB1.1 (VBUS), U1.18 (AVCC), U1.4 (VCC), U1.6 (VCC), U2.16 (VCC), U3.16 (VCC), U4.16 (VCC)
- net HAT2_PUSH: now reaches J2.3 (Pin_3)
- net HAT2_PUSH: now also J8.4 (Pin_4), RN4.4 (R4.1), U3.6 (D7)
- net HAT1_PUSH: now reaches J2.4 (Pin_4)
- net HAT1_PUSH: now also J8.3 (Pin_3), RN4.3 (R3.1), U3.5 (D6)
- new net: RP1B1.1, U1.31 (PD1)
- new net: C2.1, U1.20 (AREF)
- new net: RP1A1.1, U1.30 (PD0)
- new net: C1.1, U4.13 (~{DTR})
- new net: JUSB1.3 (D+), U4.5 (UD+)
- new net: JUSB1.2 (D-), U4.6 (UD-)
- new net BRAKE: J6.2 (Pin_2), RN1.3 (R3.1), U2.4 (D5)
- new net ENCODER_A: J4.1 (Pin_1), U1.32 (PD2)
- new net ENCODER_B: J4.2 (Pin_2), U1.1 (PD3)
- new net NC: J6.4 (Pin_4), J8.2 (Pin_2), RN1.1 (R1.1), RN4.2 (R2.1), U2.6 (D7), U3.4 (D5)
- new net PANEL_PUSH: J7.4 (Pin_4), RN3.4 (R4.1), U3.14 (D3)
- new net PINKY_PUSH: J6.3 (Pin_3), RN1.2 (R2.1), U2.5 (D6)
- new net RESET: C1.2, U1.29 (~{RESET}/PC6)
- new net RKJXT1F_CENTER: J6.1 (Pin_1), RN1.4 (R4.1), U2.3 (D4)
- new net RKJXT1F_DOWN: J5.2 (Pin_2), RN2.3 (R3.1), U2.12 (D1)
- new net RKJXT1F_LEFT: J5.3 (Pin_3), RN2.2 (R2.1), U2.13 (D2)
- new net RKJXT1F_RIGHT: J5.4 (Pin_4), RN2.1 (R1.1), U2.14 (D3)
- new net RKJXT1F_UP: J5.1 (Pin_1), RN2.4 (R4.1), U2.11 (D0)
- new net RX: RP1A1.2, U4.2 (TXD)
- new net SCL: J3.4 (Pin_4), U1.28 (PC5)
- new net SDA: J3.3 (Pin_3), U1.27 (PC4)
- new net SH_DATA2: U1.13 (PB1), U3.9 (Q7)
- new net SH_DATA3: U1.14 (PB2), U2.9 (Q7)
- new net THUMB_PUSH: J7.1 (Pin_1), RN3.1 (R1.1), U3.11 (D0)
- new net THUMB_X: J3.1 (Pin_1), U1.25 (PC2)
- new net THUMB_Y: J3.2 (Pin_2), U1.26 (PC3)
- new net TOP_SIDE_PUSH: J8.1 (Pin_1), RN4.1 (R1.1), U3.3 (D4)
- new net TRIGGER_1: J7.2 (Pin_2), RN3.2 (R2.1), U3.12 (D1)
- new net TRIGGER_2: J7.3 (Pin_3), RN3.3 (R3.1), U3.13 (D2)
- new net TX: RP1B1.2, U4.3 (RXD)
Other:
- note added: "Faceplate-PCB connectors"
- note added: "USB"
- moved on the sheet: J1, J2

Commit message: Finished preliminary routing of sub-controller pcb
Parts:
- C1: value (none) -> 100nF; footprint (none) -> Resistor_SMD:R_0201_0603Metric_Pad0.64x0.40mm_HandSolder
- J1: value (none) -> Conn_01x03_Male; footprint (none) -> Connector_PinSocket_2.54mm:PinSocket_1x03_P2.54mm_Vertical
- J2: value (none) -> Conn_01x04_Male; footprint (none) -> Connector_PinSocket_2.54mm:PinSocket_1x04_P2.54mm_Vertical
- J3, J5, J6, J7, J8: value (none) -> Conn_01x04_Female; footprint (none) -> Connector_PinSocket_2.54mm:PinSocket_1x04_P2.54mm_Vertical
- J4: value (none) -> Conn_01x02_Female; footprint (none) -> Connector_PinSocket_2.54mm:PinSocket_1x02_P2.54mm_Vertical
- JUSB1: value (none) -> USB_B_Micro; footprint (none) -> Connector_USB:USB_Micro-B_Molex_47346-0001
- RN1, RN2, RN3, RN4: value (none) -> 1k; footprint (none) -> Resistor_SMD:R_Array_Convex_4x1206
- RP1A1: value (none) -> 1k; footprint (none) -> Resistor_SMD:R_0201_0603Metric_Pad0.64x0.40mm_HandSolder
- U1: value (none) -> ATmega328P-A; footprint (none) -> Package_QFP:TQFP-32_7x7mm_P0.8mm
- U2, U3: value (none) -> 74HC165; footprint (none) -> Package_SO:TSSOP-16_4.4x5mm_P0.65mm
Connections:
- net NC renamed RESERVED1
- net RESERVED1: no longer J8.2 (Pin_2), RN4.2 (R2.1), U3.4 (D5)
- new net RESERVED2: J8.2 (Pin_2), RN4.2 (R2.1), U3.4 (D5)

Commit message: schematic changes. Bypass capacitor, I2C pullup
Parts:
- added C3, C4, C5, C6: (no value), symbol Device:C
- added J9: (no value), symbol Connector:Conn_01x02_Female
- added R1: (no value), symbol Device:R
Connections:
- net +5V: now also C3.1, C4.1, C5.1, C6.1, J9.2 (Pin_2)
- net GND: now also C3.2, C4.2, C5.2, C6.2, J9.1 (Pin_1)
- net SDA: now also R1.1
Other:
- moved on the sheet: J3

Commit message: PCB rework
Parts:
- removed JUSB1: USB_B_Micro, Connector_USB:USB_Micro-B_Molex_47346-0001, symbol Connector:USB_B_Micro
- added J10: Conn_01x04_Female, Connector_PinSocket_2.54mm:PinSocket_1x04_P2.54mm_Vertical, symbol Connector:Conn_01x04_Female
- C1: value 100nF -> (none); footprint Resistor_SMD:R_0201_0603Metric_Pad0.64x0.40mm_HandSolder -> (none)
- C2: footprint Resistor_SMD:R_0201_0603Metric_Pad0.64x0.40mm_HandSolder -> Capacitor_SMD:C_0603_1608Metric_Pad1.08x0.95mm_HandSolder
- C3, C4, C5, C6: value (none) -> 100nF; footprint (none) -> Capacitor_SMD:C_0603_1608Metric_Pad1.08x0.95mm_HandSolder
- J9: value (none) -> Conn_01x02_Female; footprint (none) -> Connector_PinSocket_2.54mm:PinSocket_1x02_P2.54mm_Vertical
- R1: value (none) -> 4.7k; footprint (none) -> Resistor_SMD:R_0603_1608Metric_Pad0.98x0.95mm_HandSolder
- RP1A1, RP1B1: footprint Resistor_SMD:R_0201_0603Metric_Pad0.64x0.40mm_HandSolder -> Resistor_SMD:R_0603_1608Metric_Pad0.98x0.95mm_HandSolder
Connections:
- net +5V: now also R1.2, J10.4 (Pin_4)
- net GND: now also J10.1 (Pin_1)
- net at U4.5 (UD+): now also J10.2 (Pin_2)
- net at U4.6 (UD-): now also J10.3 (Pin_3)

Commit message: Some PCB changes
Parts:
- added C7: 4.7nF, Capacitor_SMD:C_0603_1608Metric_Pad1.08x0.95mm_HandSolder, symbol Device:C
- C1: value (none) -> 100nF; footprint (none) -> Resistor_SMD:R_0603_1608Metric_Pad0.98x0.95mm_HandSolder
- U4: value CH340G -> CH340C
Connections:
- net +5V: no longer C6.1, J10.4 (Pin_4), U4.16 (VCC)
- net GND: now also C7.1
- net at U4.4 (V3): now also C7.2
- new net: C6.1, J10.4 (Pin_4), U4.16 (VCC)
Changed lines of the file:
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@@
   (junction (at 50.8 29.21) (diameter 0) (color 0 0 0 0)
   )
+  (junction (at 114.3 128.27) (diameter 0) (color 0 0 0 0)
+  )
   (junction (at 223.52 116.84) (diameter 0) (color 0 0 0 0)
   )
@@
     (stroke (width 0) (type default) (color 0 0 0 0))
   )
+  (wire (pts (xy 121.92 121.92) (xy 133.35 121.92))
+    (stroke (width 0) (type default) (color 0 0 0 0))
+  )
   (wire (pts (xy 226.06 102.87) (xy 240.03 102.87))
     (stroke (width 0) (type default) (color 0 0 0 0))
@@
     (stroke (width 0) (type default) (color 0 0 0 0))
   )
+  (wire (pts (xy 114.3 128.27) (xy 114.3 132.08))
+    (stroke (width 0) (type default) (color 0 0 0 0))
+  )
   (wire (pts (xy 224.79 101.6) (xy 237.49 101.6))
     (stroke (width 0) (type default) (color 0 0 0 0))
@@
     (stroke (width 0) (type default) (color 0 0 0 0))
   )
-  (wire (pts (xy 114.3 118.11) (xy 114.3 124.46))
+  (wire (pts (xy 114.3 118.11) (xy 114.3 128.27))
     (stroke (width 0) (type default) (color 0 0 0 0))
   )
@@
     (stroke (width 0) (type default) (color 0 0 0 0))
   )
-  (wire (pts (xy 133.35 125.73) (xy 133.35 127))
+  (wire (pts (xy 133.35 121.92) (xy 133.35 127))
     (stroke (width 0) (type default) (color 0 0 0 0))
   )
@@
     (stroke (width 0) (type default) (color 0 0 0 0))
   )
-  (wire (pts (xy 121.92 127) (xy 133.35 127))
-    (stroke (width 0) (type default) (color 0 0 0 0))
-  )
   (wire (pts (xy 209.55 46.99) (xy 254 46.99))
     (stroke (width 0) (type default) (color 0 0 0 0))
@@
     (stroke (width 0) (type default) (color 0 0 0 0))
   )
-  (wire (pts (xy 121.92 118.11) (xy 121.92 127))
+  (wire (pts (xy 121.92 118.11) (xy 121.92 121.92))
     (stroke (width 0) (type default) (color 0 0 0 0))
   )
@@
     (stroke (width 0) (type default) (color 0 0 0 0))
   )
+  (wire (pts (xy 128.27 128.27) (xy 130.81 128.27))
+    (stroke (width 0) (type default) (color 0 0 0 0))
+  )
   (wire (pts (xy 66.04 19.05) (xy 74.93 19.05))
     (stroke (width 0) (type default) (color 0 0 0 0))
@@
     (stroke (width 0) (type default) (color 0 0 0 0))
   )
+  (wire (pts (xy 114.3 128.27) (xy 120.65 128.27))
+    (stroke (width 0) (type default) (color 0 0 0 0))
+  )
   (wire (pts (xy 66.04 26.67) (xy 74.93 26.67))
     (stroke (width 0) (type default) (color 0 0 0 0))
@@
   )
   (wire (pts (xy 212.09 26.67) (xy 212.09 44.45))
+    (stroke (width 0) (type default) (color 0 0 0 0))
+  )
+  (wire (pts (xy 130.81 128.27) (xy 130.81 129.54))
     (stroke (width 0) (type default) (color 0 0 0 0))
   )
@@
       (effects (font (size 1.27 1.27)) (justify left))
     )
-    (property "Value" "CH340G" (id 1) (at 135.3694 162.56 0)
+    (property "Value" "CH340C" (id 1) (at 135.3694 162.56 0)
       (effects (font (size 1.27 1.27)) (justify left))
     )
@@
     (in_bom yes) (on_board yes) (fields_autoplaced)
     (property "Reference" "C1" (id 0) (at 151.13 144.78 90))
-    (property "Value" "" (id 1) (at 151.13 147.32 90))
-    (property "Footprint" "" (id 2) (at 154.94 151.4348 0)
+    (property "Value" "100nF" (id 1) (at 151.13 147.32 90))
+    (property "Footprint" "Resistor_SMD:R_0603_1608Metric_Pad0.98x0.95mm_HandSolder" (id 2) (at 154.94 151.4348 0)
       (effects (font (size 1.27 1.27)) hide)
     )
@@
     (pin "4")
   )
-  (symbol (lib_id "power:GND") (at 114.3 124.46 0) (unit 1)
-    (in_bom yes) (on_board yes) (fields_autoplaced)
-    (property "Reference" "#PWR0111" (id 0) (at 114.3 130.81 0)
-      (effects (font (size 1.27 1.27)) hide)
-    )
-    (property "Value" "GND" (id 1) (at 114.3 129.54 0))
-    (property "Footprint" "" (id 2) (at 114.3 124.46 0)
-      (effects (font (size 1.27 1.27)) hide)
-    )
-    (property "Datasheet" "" (id 3) (at 114.3 124.46 0)
+  (symbol (lib_id "power:GND") (at 114.3 132.08 0) (unit 1)
+    (in_bom yes) (on_board yes) (fields_autoplaced)
+    (property "Reference" "#PWR0111" (id 0) (at 114.3 138.43 0)
+      (effects (font (size 1.27 1.27)) hide)
+    )
+    (property "Value" "GND" (id 1) (at 114.3 137.16 0))
+    (property "Footprint" "" (id 2) (at 114.3 132.08 0)
+      (effects (font (size 1.27 1.27)) hide)
+    )
+    (property "Datasheet" "" (id 3) (at 114.3 132.08 0)
       (effects (font (size 1.27 1.27)) hide)
     )
@@
     (pin "1")
   )
+  (symbol (lib_id "Device:C") (at 124.46 128.27 90) (unit 1)
+    (in_bom yes) (on_board yes)
+    (property "Reference" "C7" (id 0) (at 121.92 129.54 90))
+    (property "Value" "4.7nF" (id 1) (at 124.46 124.46 90))
+    (property "Footprint" "Capacitor_SMD:C_0603_1608Metric_Pad1.08x0.95mm_HandSolder" (id 2) (at 128.27 127.3048 0)
+      (effects (font (size 1.27 1.27)) hide)
+    )
+    (property "Datasheet" "~" (id 3) (at 124.46 128.27 0)
+      (effects (font (size 1.27 1.27)) hide)
+    )
+    (pin "1")
+    (pin "2")
+  )
   (symbol (lib_id "power:GND") (at 96.52 44.45 0) (unit 1)
     (in_bom yes) (on_board yes) (fields_autoplaced)
@@
     (pin "4")
   )
-  (symbol (lib_id "power:+5V") (at 133.35 125.73 0) (unit 1)
-    (in_bom yes) (on_board yes) (fields_autoplaced)
-    (property "Reference" "#PWR0112" (id 0) (at 133.35 129.54 0)
-      (effects (font (size 1.27 1.27)) hide)
-    )
-    (property "Value" "+5V" (id 1) (at 133.35 120.65 0))
-    (property "Footprint" "" (id 2) (at 133.35 125.73 0)
-      (effects (font (size 1.27 1.27)) hide)
-    )
-    (property "Datasheet" "" (id 3) (at 133.35 125.73 0)
-      (effects (font (size 1.27 1.27)) hide)
-    )
-    (pin "1")
-  )
   (symbol (lib_id "power:GND") (at 210.82 147.32 0) (unit 1)
     (in_bom yes) (on_board yes) (fields_autoplaced)
@@
       (reference "#PWR0111") (unit 1) (value "GND") (footprint "")
     )
-    (path "/f75975ee-c51a-47d0-8e14-93c9d5060fca"
-      (reference "#PWR0112") (unit 1) (value "+5V") (footprint "")
-    )
     (path "/85eabc02-7208-4303-be09-8609ef868e11"
       (reference "#PWR0113") (unit 1) (value "+5V") (footprint "")
@@
       (reference "C6") (unit 1) (value "100nF") (footprint "Capacitor_SMD:C_0603_1608Metric_Pad1.08x0.95mm_HandSolder")
     )
+    (path "/c59f7c10-88c3-41b5-893e-0e94f3460030"
+      (reference "C7") (unit 1) (value "4.7nF") (footprint "Capacitor_SMD:C_0603_1608Metric_Pad1.08x0.95mm_HandSolder")
+    )
     (path "/7fb65ec1-ece3-48e1-bdf5-4413b4bf1f25"
       (reference "J1") (unit 1) (value "Conn_01x03_Male") (footprint "Connector_PinSocket_2.54mm:PinSocket_1x03_P2.54mm_Vertical")
@@
     )
     (path "/6b6ca22f-7349-4186-9d31-1c8789b33c55"
-      (reference "U4") (unit 1) (value "CH340G") (footprint "Package_SO:SOIC-16_3.9x9.9mm_P1.27mm")
-    )
-  )
+      (reference "U4") (unit 1) (value "CH340C") (footprint "Package_SO:SOIC-16_3.9x9.9mm_P1.27mm")
+    )
+  )
